File: Hardware/Apo Board 2017 ATmega328.sch (EAGLE design)
At the start: 16 parts, among them U3 LED-TRICOLOR-5050-IC, U4 LED-TRICOLOR-5050-IC, U5 LED-TRICOLOR-5050-IC, U6 LED-TRICOLOR-5050-IC, U7 LED-TRICOLOR-5050-IC

Commit message: ATMega328 Version
Parts:
- added C5: 4.7uF, SparkFun-Passives:CAPKIT
- added C6: 0.1uF, SparkFun-Passives:CAPKIT
- added LED1: (no value), SparkFun-LED:LED5MM
- added R1: 10k, SparkFun-Resistors:RESISTORPTH-1/4W
- added R5: 20K, SparkFun-Passives:RESISTORKIT
- added U1, U10, U11, U8, U9: LED-TRICOLOR-5050-IC, SparkFun-LED:LED-TRICOLOR-5050-IC
- added X1: 16Mhz, 1_Dan Master:CERAMIC_RESONATOR
- C1: value (none) -> 1000uF
- JP1: device SparkFun-Connectors:M04PTH -> SparkFun-Connectors:M03PTH
- JP2: value (none) -> ISP; device SparkFun-Connectors:M04PTH -> SparkFun:AVR_SPI_PRG_6PTH
- JP4: value (none) -> FTDI_BASICPTH; device SparkFun-Connectors:M031X03_NO_SILK -> SparkFun-Connectors:FTDI_BASICPTH
- U2: value (none) -> ATMEGA328P_PDIP; device SparkFun-PowerIC:MIC52055V -> SparkFun-DigitalIC:ATMEGA328P_PDIP
Connections:
- removed net 2: JP1.2, JP4.3
- removed net 3: JP1.3, JP4.2
- removed net RST: JP1.1
- new net +5V: C5.1, JP1.1, JP2.2, JP4.4, R5.2, U1.VDD, U10.VDD, U11.VDD, U2.AREF, U2.AVCC, U2.VCC, U3.VDD, U4.VDD, U5.VDD, U6.VDD, U7.VDD, U8.VDD, U9.VDD
- new net BUTTON_PIN: S2.1, S2.2, U2.PD2(INT0)
- new net DOUT_DIN: U11.DI, U4.DO
- new net DTR: C6.1, JP4.1
- new net IR_RECEIVE: JP1.3
- new net IR_SEND: R1.1
- new net LED_PIN: U7.DI
- new net N$10: C6.2, R5.1, U2.PC6(/RESET)
- new net N$11: U10.DO, U9.DI
- new net N$12: U2.PD3(INT1)
- new net N$13: U1.DI, U9.DO
- new net N$14: U1.DO, U8.DI
- new net N$15: U2.PD4(XCK/T0)
- new net N$16: U2.PD5(T1)
- new net N$17: U2.PD6(AIN0)
- new net N$18: U2.PD7(AIN1)
- new net N$19: U2.PB0(ICP)
- new net N$20: U2.PB1(OC1A)
- new net N$21: U2.PB2(SS/OC1B)
- new net N$22: U2.PC5(ADC5/SCL)
- new net N$23: U2.PC4(ADC4/SDA)
- new net N$24: U2.PC3(ADC3)
- new net N$25: U2.PC2(ADC2)
- new net N$26: U2.PC1(ADC1)
- new net N$27: U2.PC0(ADC0)
- new net N$3: LED1.A, R1.2
- new net N$4: U2.PB6(XTAL1/TOSC1), X1.P$1
- new net N$7: U2.PB7(XTAL2/TOSC2), X1.P$3
- new net N$9: U10.DI, U11.DO
- new net RESET: JP2.5
- new net RX: JP4.3, U2.PD0(RXD)
- new net TX: JP4.2, U2.PD1(TXD)
- net GND: now also C5.2, JP1.2, JP2.6, JP4.5, JP4.6, LED1.C, S2.3, S2.4, U1.VSS, U10.VSS, U11.VSS, U2.GND@1, U2.GND@2, U8.VSS, U9.VSS, X1.P$2; no longer JP1.4, JP4.1, S2.1, S2.2, U2.GND
- net MISO: now also JP2.1, U2.PB4(MISO); no longer JP2.2, S2.3, S2.4
- net MOSI: now also JP2.4, U2.PB3(MOSI/OC2); no longer JP2.1, U7.DI
- net SCK: now also U2.PB5(SCK)
- net VCC: no longer JP2.4, U2.OUT, U3.VDD, U4.VDD, U5.VDD, U6.VDD, U7.VDD
- net VREG: no longer U2.EN, U2.IN
Other:
- note removed: "DIP socket"
- note removed: "for ATtiny45/85"
- moved on the sheet: 0.1UF, C1, C3, JP3, S2
