File: Hardware/Apo Board 2017_large.brd (EAGLE design)
At the start: 69.8 x 43.2 mm, 19 parts, among them U3 LED-TRICOLOR-5050-IC, U4 LED-TRICOLOR-5050-IC, U5 LED-TRICOLOR-5050-IC, U6 LED-TRICOLOR-5050-IC, U7 LED-TRICOLOR-5050-IC

Commit message: ATMega328 Version
Parts:
- removed R1: PHOTOCELLPTH, SparkFun-Sensors:PHOTOCELL
- removed R2, R3: 10k, SparkFun-Resistors:AXIAL-0.4
- moved U4 2.93 mm to (-9.09, 3.48)
- moved U7 2.75 mm to (-5.92, -7.32)
- moved U6 2.70 mm to (6.53, -6.81)
- moved U5 2.40 mm to (8.43, 3.86)
- moved U3 2.04 mm to (-0.08, 9.07)
Connections:
- net GND: no longer R2.P$1
- net MISO: no longer R3.P$1
- net SCK: no longer R1.2, R2.P$2
- net VCC: no longer R1.1, R3.P$2
Routing:
- net N$6: track 15.4 -> 19.7 mm
- net N$2: track 8.41 -> 12.4 mm
- net N$1: track 5.08 -> 8.65 mm
- net N$5: track 17.8 -> 15.4 mm
