File: Hardware/Apo Board 2017 ATmega328SMD_PAM2401.sch (EAGLE design)
At the start: 38 parts, among them Q1 RESONATORSMD, U1 LED-TRICOLOR-5050-IC, U10 LED-TRICOLOR-5050-IC, U11 LED-TRICOLOR-5050-IC, U13 ATMEGA328, U2 PAM2401, U3 LED-TRICOLOR-5050-IC, U4 LED-TRICOLOR-5050-IC, U5 LED-TRICOLOR-5050-IC, U6 LED-TRICOLOR-5050-IC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

Commit message: Added Deacon board files. finished prelim layout
Connections:
- net BUTTON: now also U13.PD2(INT0); no longer U13.PB2(SS/OC1B)
- net IR_RX: now also U13.PB0(ICP); no longer U13.PB1(OC1A)
- net IR_TX: now also U13.PB1(OC1A); no longer U13.PB0(ICP)
Changed lines of the file:
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@@
 <net name="BUTTON" class="0">
-<segment>
-<wire x1="91.44" y1="15.24" x2="109.22" y2="15.24" width="0.1524" layer="91"/>
-<label x="109.22" y="15.24" size="1.27" layer="95" xref="yes"/>
-<pinref part="U13" gate="G$1" pin="PB2(SS/OC1B)"/>
-</segment>
 <segment>
 <pinref part="S2" gate="S" pin="1"/>
@@
 <junction x="165.1" y="104.14"/>
 <label x="162.56" y="104.14" size="1.27" layer="95" rot="R180" xref="yes"/>
+</segment>
+<segment>
+<pinref part="U13" gate="G$1" pin="PD2(INT0)"/>
+<wire x1="91.44" y1="38.1" x2="106.68" y2="38.1" width="0.1524" layer="91"/>
+<label x="106.68" y="38.1" size="1.27" layer="95" xref="yes"/>
 </segment>
 </net>
@@
 <net name="IR_TX" class="0">
 <segment>
-<pinref part="U13" gate="G$1" pin="PB0(ICP)"/>
-<wire x1="91.44" y1="20.32" x2="93.98" y2="20.32" width="0.1524" layer="91"/>
-<label x="93.98" y="20.32" size="1.27" layer="95" xref="yes"/>
-</segment>
-<segment>
 <pinref part="R1" gate="G$1" pin="1"/>
 <wire x1="236.22" y1="121.92" x2="236.22" y2="124.46" width="0.1524" layer="91"/>
@@
 <label x="233.68" y="124.46" size="1.27" layer="95" rot="R180" xref="yes"/>
 </segment>
-</net>
-<net name="IR_RX" class="0">
 <segment>
 <pinref part="U13" gate="G$1" pin="PB1(OC1A)"/>
@@
 <label x="93.98" y="17.78" size="1.27" layer="95" xref="yes"/>
 </segment>
+</net>
+<net name="IR_RX" class="0">
 <segment>
 <pinref part="JP1" gate="G$1" pin="3"/>
@@
 <label x="205.74" y="104.14" size="1.27" layer="95" rot="R180" xref="yes"/>
 </segment>
+<segment>
+<pinref part="U13" gate="G$1" pin="PB0(ICP)"/>
+<wire x1="91.44" y1="20.32" x2="93.98" y2="20.32" width="0.1524" layer="91"/>
+<label x="93.98" y="20.32" size="1.27" layer="95" xref="yes"/>
+</segment>
 </net>

Commit message: Final touches before review
Parts:
- added C6: (no value), SparkFun-Capacitors:CAPPTH
- added R3: 100k, SparkFun-Resistors:10K-1%RES-00824
Connections:
- new net N$4: R3.2, U2.RSET
- net +5V: now also C6.1
- net GND: now also C6.2, R3.1
- net N$10: now also U2.EN
Other:
- note added: "DNP R3: leaving pad in case adjustments are needed for the inductor on prototype"
- note added: "Marshall thinks we still need a large capacitor for the outout of the step up. Leaving here for SMD or PTH addition to prototype"
- note added: "V0.1"
- note removed: "DIODE HERE??"
Changed lines of the file:
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@@
 <part name="GND17" library="SparkFun" deviceset="GND" device=""/>
 <part name="GND21" library="SparkFun" deviceset="GND" device=""/>
+<part name="R3" library="SparkFun-Resistors" deviceset="10K-1%" device="RES-00824" value="100k"/>
+<part name="GND23" library="SparkFun" deviceset="GND" device=""/>
+<part name="P+16" library="supply1" deviceset="+5V" device=""/>
+<part name="GND24" library="SparkFun" deviceset="GND" device=""/>
+<part name="C6" library="SparkFun-Capacitors" deviceset="CAP" device="PTH"/>
 </parts>
 <sheets>
@@
 <plain>
 <text x="166.37" y="11.43" size="2.54" layer="94">Joel Bartlett</text>
-<text x="81.28" y="124.46" size="1.27" layer="91">DIODE HERE??</text>
 <wire x1="0" y1="137.16" x2="0" y2="134.62" width="0.2032" layer="94" style="shortdash"/>
 <wire x1="0" y1="134.62" x2="147.32" y2="134.62" width="0.2032" layer="94" style="shortdash"/>
@@
 <text x="53.34" y="81.28" size="2.54" layer="97">ATMEGA328P-AU</text>
 <text x="172.72" y="81.28" size="2.54" layer="97">ATMEGA328P Programming</text>
+<text x="12.192" y="90.17" size="1.27" layer="91">DNP R3: leaving pad in case adjustments
+ are needed for the inductor on prototype</text>
+<text x="116.84" y="99.06" size="1.27" layer="91">Marshall thinks we still need a large
+ capacitor for the outout of the step up.
+Leaving here for SMD or PTH addition
+to prototype</text>
+<text x="237.49" y="6.35" size="2.54" layer="94">V0.1</text>
 </plain>
 <instances>
@@
 <attribute name="VALUE" x="27.94" y="40.64" size="1.778" layer="96" rot="R270"/>
 </instance>
+<instance part="R3" gate="G$1" x="48.26" y="93.98" rot="R90"/>
+<instance part="GND23" gate="1" x="48.26" y="83.82" rot="MR0"/>
+<instance part="P+16" gate="1" x="111.76" y="119.38"/>
+<instance part="GND24" gate="1" x="111.76" y="101.6" rot="MR0"/>
+<instance part="C6" gate="G$1" x="111.76" y="109.22"/>
 </instances>
 <busses>
@@
 <pinref part="Q1" gate="G$1" pin="2"/>
 <pinref part="GND21" gate="1" pin="GND"/>
+</segment>
+<segment>
+<pinref part="R3" gate="G$1" pin="1"/>
+<pinref part="GND23" gate="1" pin="GND"/>
+<wire x1="48.26" y1="86.36" x2="48.26" y2="88.9" width="0.1524" layer="91"/>
+</segment>
+<segment>
+<pinref part="GND24" gate="1" pin="GND"/>
+<wire x1="111.76" y1="104.14" x2="111.76" y2="106.68" width="0.1524" layer="91"/>
+<pinref part="C6" gate="G$1" pin="2"/>
 </segment>
 </net>
@@
 <junction x="93.98" y="121.92"/>
 </segment>
+<segment>
+<pinref part="P+16" gate="1" pin="+5V"/>
+<wire x1="111.76" y1="114.3" x2="111.76" y2="116.84" width="0.1524" layer="91"/>
+<pinref part="C6" gate="G$1" pin="1"/>
+</segment>
 </net>
 <net name="TX" class="0">
@@
 <junction x="43.18" y="119.38"/>
 <pinref part="C2" gate="G$1" pin="1"/>
+<pinref part="U2" gate="G$1" pin="EN"/>
+<wire x1="50.8" y1="104.14" x2="48.26" y2="104.14" width="0.1524" layer="91"/>
+<wire x1="48.26" y1="104.14" x2="48.26" y2="119.38" width="0.1524" layer="91"/>
 </segment>
 </net>
@@
 </segment>
 </net>
+<net name="N$4" class="0">
+<segment>
+<pinref part="U2" gate="G$1" pin="RSET"/>
+<pinref part="R3" gate="G$1" pin="2"/>
+<wire x1="50.8" y1="99.06" x2="48.26" y2="99.06" width="0.1524" layer="91"/>
+</segment>
+</net>

Commit message: Final version for Prototypes V0.1 and GERBERS
Parts:
- C6: device SparkFun-Capacitors:CAPPTH -> SparkFun-Capacitors:CAP1206
- U1: value LED-TRICOLOR-5050-IC -> PAM2401; device SparkFun-LED:LED-TRICOLOR-5050-IC -> SparkFun-PowerIC:PAM2401
- U2: value PAM2401 -> LED-TRICOLOR-5050-IC; device SparkFun-PowerIC:PAM2401 -> SparkFun-LED:LED-TRICOLOR-5050-IC
- renumbered JP1 to U12
Connections:
- net N$7 renamed +BATT_RAW
- net +5V: now also U1.OUT, U2.VDD; no longer U1.VDD, U2.OUT
- net GND: now also U1.AGND, U1.PGND, U2.VSS; no longer U1.VSS, U2.AGND, U2.PGND
- net N$10: now also U1.EN, U1.VIN; no longer U2.EN, U2.VIN
- net N$12: now also U1.FB; no longer U2.FB
- net N$13: now also U2.DI; no longer U1.DI
- net N$14: now also U2.DO; no longer U1.DO
- net N$4: now also U1.RSET; no longer U2.RSET
- net N$8: now also U1.LX; no longer U2.LX
Changed lines of the file:
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@@
 <setting verticaltext="up"/>
 </settings>
-<grid distance="0.1" unitdist="inch" unit="inch" style="lines" multiple="1" display="no" altdistance="0.01" altunitdist="inch" altunit="inch"/>
+<grid distance="0.05" unitdist="inch" unit="inch" style="lines" multiple="1" display="yes" altdistance="0.005" altunitdist="inch" altunit="inch"/>
 <layers>
 <layer number="1" name="Top" color="4" fill="1" visible="no" active="no"/>
@@
 <part name="GND15" library="supply1" deviceset="GND" device=""/>
 <part name="JP4" library="SparkFun-Connectors" deviceset="FTDI_BASIC" device="PTH"/>
-<part name="U1" library="SparkFun-LED" deviceset="LED-TRICOLOR-5050-IC" device=""/>
+<part name="U2" library="SparkFun-LED" deviceset="LED-TRICOLOR-5050-IC" device=""/>
 <part name="U8" library="SparkFun-LED" deviceset="LED-TRICOLOR-5050-IC" device=""/>
 <part name="U9" library="SparkFun-LED" deviceset="LED-TRICOLOR-5050-IC" device=""/>
@@
 <part name="GND16" library="SparkFun-Aesthetics" deviceset="GND" device=""/>
 <part name="GND18" library="SparkFun-Aesthetics" deviceset="GND" device=""/>
-<part name="JP1" library="SparkFun-Connectors" deviceset="M03" device="IR_RECEIVER"/>
+<part name="U12" library="SparkFun-Connectors" deviceset="M03" device="IR_RECEIVER"/>
 <part name="P+2" library="supply1" deviceset="+5V" device=""/>
 <part name="P+3" library="supply1" deviceset="+5V" device=""/>
@@
 <part name="TP6" library="SparkFun-Passives" deviceset="TEST-POINT" device="3X5" value="TP-3x5"/>
 <part name="P+18" library="supply1" deviceset="+5V" device=""/>
-<part name="U2" library="SparkFun-PowerIC" deviceset="PAM2401" device=""/>
+<part name="U1" library="SparkFun-PowerIC" deviceset="PAM2401" device=""/>
 <part name="L1" library="SparkFun-Passives" deviceset="INDUCTOR" device="CR54" value="2.2uH"/>
 <part name="GND7" library="SparkFun" deviceset="GND" device=""/>
@@
 <part name="P+16" library="supply1" deviceset="+5V" device=""/>
 <part name="GND24" library="SparkFun" deviceset="GND" device=""/>
-<part name="C6" library="SparkFun-Capacitors" deviceset="CAP" device="PTH"/>
+<part name="C6" library="SparkFun-Capacitors" deviceset="CAP" device="1206"/>
 </parts>
 <sheets>
@@
 <text x="53.34" y="81.28" size="2.54" layer="97">ATMEGA328P-AU</text>
 <text x="172.72" y="81.28" size="2.54" layer="97">ATMEGA328P Programming</text>
-<text x="12.192" y="90.17" size="1.27" layer="91">DNP R3: leaving pad in case adjustments
+<text x="9.652" y="90.17" size="1.27" layer="91">DNP R3: leaving pad in case adjustments
  are needed for the inductor on prototype</text>
 <text x="116.84" y="99.06" size="1.27" layer="91">Marshall thinks we still need a large
@@
 <instance part="GND15" gate="1" x="170.18" y="50.8"/>
 <instance part="JP4" gate="G$1" x="182.88" y="63.5" rot="R180"/>
-<instance part="U1" gate="U1" x="162.56" y="149.86"/>
+<instance part="U2" gate="U1" x="162.56" y="149.86"/>
 <instance part="U8" gate="U1" x="200.66" y="149.86"/>
 <instance part="U9" gate="U1" x="124.46" y="149.86"/>
@@
 <instance part="GND16" gate="1" x="177.8" y="149.86"/>
 <instance part="GND18" gate="1" x="215.9" y="149.86"/>
-<instance part="JP1" gate="G$1" x="218.44" y="106.68" rot="R180"/>
+<instance part="U12" gate="G$1" x="218.44" y="106.68" rot="R180"/>
 <instance part="P+2" gate="1" x="27.94" y="160.02"/>
 <instance part="P+3" gate="1" x="68.58" y="160.02"/>
@@
 </instance>
 <instance part="GND38" gate="1" x="40.64" y="5.08"/>
-<instance part="P+1" gate="1" x="40.64" y="76.2"/>
+<instance part="P+1" gate="1" x="33.02" y="60.96" rot="R90"/>
 <instance part="GND22" gate="1" x="27.94" y="99.06" rot="MR0"/>
 <instance part="S1" gate="1" x="35.56" y="121.92" rot="MR180"/>
@@
 </instance>
 <instance part="P+18" gate="1" x="226.06" y="73.66"/>
-<instance part="U2" gate="G$1" x="63.5" y="109.22"/>
+<instance part="U1" gate="G$1" x="63.5" y="109.22"/>
 <instance part="L1" gate="G$1" x="63.5" y="127" rot="R90"/>
 <instance part="GND7" gate="1" x="43.18" y="104.14" rot="MR0"/>
@@
 <segment>
 <pinref part="GND16" gate="1" pin="GND"/>
-<pinref part="U1" gate="U1" pin="VSS"/>
+<pinref part="U2" gate="U1" pin="VSS"/>
 <wire x1="177.8" y1="152.4" x2="177.8" y2="154.94" width="0.1524" layer="91"/>
 <wire x1="177.8" y1="154.94" x2="175.26" y2="154.94" width="0.1524" layer="91"/>
@@
 </segment>
 <segment>
-<pinref part="JP1" gate="G$1" pin="2"/>
+<pinref part="U12" gate="G$1" pin="2"/>
 <pinref part="GND19" gate="1" pin="GND"/>
 <wire x1="210.82" y1="106.68" x2="208.28" y2="106.68" width="0.1524" layer="91"/>
@@
 </segment>
 <segment>
-<pinref part="U2" gate="G$1" pin="AGND"/>
+<pinref part="U1" gate="G$1" pin="AGND"/>
 <pinref part="GND10" gate="1" pin="GND"/>
 <wire x1="76.2" y1="104.14" x2="78.74" y2="104.14" width="0.1524" layer="91"/>
 <wire x1="78.74" y1="104.14" x2="78.74" y2="99.06" width="0.1524" layer="91"/>
-<pinref part="U2" gate="G$1" pin="PGND"/>
+<pinref part="U1" gate="G$1" pin="PGND"/>
 <wire x1="78.74" y1="99.06" x2="78.74" y2="96.52" width="0.1524" layer="91"/>
 <wire x1="76.2" y1="99.06" x2="78.74" y2="99.06" width="0.1524" layer="91"/>
@@
 </segment>
 <segment>
-<pinref part="U1" gate="U1" pin="VDD"/>
+<pinref part="U2" gate="U1" pin="VDD"/>
 <wire x1="144.78" y1="157.48" x2="144.78" y2="154.94" width="0.1524" layer="91"/>
 <wire x1="144.78" y1="154.94" x2="147.32" y2="154.94" width="0.1524" layer="91"/>
@@
 </segment>
 <segment>
-<pinref part="JP1" gate="G$1" pin="1"/>
+<pinref part="U12" gate="G$1" pin="1"/>
 <pinref part="P+15" gate="1" pin="+5V"/>
 <wire x1="210.82" y1="109.22" x2="208.28" y2="109.22" width="0.1524" layer="91"/>
@@
 <wire x1="40.64" y1="55.88" x2="40.64" y2="58.42" width="0.1524" layer="91"/>
 <wire x1="40.64" y1="58.42" x2="40.64" y2="60.96" width="0.1524" layer="91"/>
-<wire x1="40.64" y1="60.96" x2="40.64" y2="73.66" width="0.1524" layer="91"/>
+<wire x1="40.64" y1="60.96" x2="35.56" y2="60.96" width="0.1524" layer="91"/>
 <wire x1="43.18" y1="58.42" x2="40.64" y2="58.42" width="0.1524" layer="91"/>
 <wire x1="43.18" y1="60.96" x2="40.64" y2="60.96" width="0.1524" layer="91"/>
@@
 </segment>
 <segment>
-<pinref part="U2" gate="G$1" pin="OUT"/>
+<pinref part="U1" gate="G$1" pin="OUT"/>
 <wire x1="76.2" y1="114.3" x2="81.28" y2="114.3" width="0.1524" layer="91"/>
 <wire x1="81.28" y1="114.3" x2="81.28" y2="121.92" width="0.1524" layer="91"/>
@@
 <segment>
 <pinref part="U9" gate="U1" pin="DO"/>
-<pinref part="U1" gate="U1" pin="DI"/>
+<pinref part="U2" gate="U1" pin="DI"/>
 <wire x1="137.16" y1="147.32" x2="147.32" y2="147.32" width="0.1524" layer="91"/>
 </segment>
@@
 <net name="N$14" class="0">
 <segment>
-<pinref part="U1" gate="U1" pin="DO"/>
+<pinref part="U2" gate="U1" pin="DO"/>
 <pinref part="U8" gate="U1" pin="DI"/>
 <wire x1="175.26" y1="147.32" x2="185.42" y2="147.32" width="0.1524" layer="91"/>
@@
 <wire x1="71.12" y1="127" x2="78.74" y2="127" width="0.1524" layer="91"/>
 <wire x1="78.74" y1="127" x2="78.74" y2="119.38" width="0.1524" layer="91"/>
-<pinref part="U2" gate="G$1" pin="LX"/>
+<pinref part="U1" gate="G$1" pin="LX"/>
 <wire x1="78.74" y1="119.38" x2="76.2" y2="119.38" width="0.1524" layer="91"/>
 </segment>
@@
 <wire x1="55.88" y1="127" x2="48.26" y2="127" width="0.1524" layer="91"/>
 <wire x1="48.26" y1="127" x2="48.26" y2="119.38" width="0.1524" layer="91"/>
-<pinref part="U2" gate="G$1" pin="VIN"/>
+<pinref part="U1" gate="G$1" pin="VIN"/>
 <wire x1="48.26" y1="119.38" x2="50.8" y2="119.38" width="0.1524" layer="91"/>
 <pinref part="S1" gate="1" pin="O"/>
@@
 <junction x="43.18" y="119.38"/>
 <pinref part="C2" gate="G$1" pin="1"/>
-<pinref part="U2" gate="G$1" pin="EN"/>
+<pinref part="U1" gate="G$1" pin="EN"/>
 <wire x1="50.8" y1="104.14" x2="48.26" y2="104.14" width="0.1524" layer="91"/>
 <wire x1="48.26" y1="104.14" x2="48.26" y2="119.38" width="0.1524" layer="91"/>
@@
 <net name="N$12" class="0">
 <segment>
-<pinref part="U2" gate="G$1" pin="FB"/>
+<pinref part="U1" gate="G$1" pin="FB"/>
 <pinref part="R4" gate="G$1" pin="1"/>
 <wire x1="76.2" y1="109.22" x2="86.36" y2="109.22" width="0.1524" layer="91"/>
@@
 </segment>
 </net>
-<net name="N$7" class="0">
+<net name="+BATT_RAW" class="0">
 <segment>
 <pinref part="S1" gate="1" pin="P"/>
@@
 <net name="IR_RX" class="0">
 <segment>
-<pinref part="JP1" gate="G$1" pin="3"/>
+<pinref part="U12" gate="G$1" pin="3"/>
 <wire x1="210.82" y1="104.14" x2="205.74" y2="104.14" width="0.1524" layer="91"/>
 <label x="205.74" y="104.14" size="1.27" layer="95" rot="R180" xref="yes"/>
@@
 <net name="N$4" class="0">
 <segment>
-<pinref part="U2" gate="G$1" pin="RSET"/>
+<pinref part="U1" gate="G$1" pin="RSET"/>
 <pinref part="R3" gate="G$1" pin="2"/>
 <wire x1="50.8" y1="99.06" x2="48.26" y2="99.06" width="0.1524" layer="91"/>
