File: Hardware/Apo Board 2017 ATmega328SMD_PAM2401.sch (EAGLE design)
At the start: 40 parts, among them Q1 RESONATORSMD, U1 PAM2401, U10 LED-TRICOLOR-5050-ICWS2812-TH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, U11 LED-TRICOLOR-5050-ICWS2812-TH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, U13 ATMEGA328, U2 LED-TRICOLOR-5050-ICWS2812-TH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, U3 LED-TRICOLOR-5050-ICWS2812-TH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, U4 LED-TRICOLOR-5050-ICWS2812-TH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, U5 LED-TRICOLOR-5050-ICWS2812-TH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, U6 LED-TRICOLOR-5050-ICWS2812-TH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

Commit message: Updating Battery footprint
Changed lines of the file:
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@@
 </classes>
 <parts>
-<part name="U3" library="SparkFun-LED" deviceset="LED-TRICOLOR-5050-IC" device="WS2812-THRU-KIT" value=""/>
-<part name="U4" library="SparkFun-LED" deviceset="LED-TRICOLOR-5050-IC" device="WS2812-THRU-KIT" value=""/>
-<part name="U5" library="SparkFun-LED" deviceset="LED-TRICOLOR-5050-IC" device="WS2812-THRU-KIT" value=""/>
-<part name="U6" library="SparkFun-LED" deviceset="LED-TRICOLOR-5050-IC" device="WS2812-THRU-KIT" value=""/>
-<part name="U7" library="SparkFun-LED" deviceset="LED-TRICOLOR-5050-IC" device="WS2812-THRU-KIT" value=""/>
+<part name="U3" library="SparkFun-LED" deviceset="LED-TRICOLOR-5050-IC" device="WS2812-THRU-KIT" value="LED-TRICOLOR-5050-ICWS2812-THRU-KIT"/>
+<part name="U4" library="SparkFun-LED" deviceset="LED-TRICOLOR-5050-IC" device="WS2812-THRU-KIT" value="LED-TRICOLOR-5050-ICWS2812-THRU-KIT"/>
+<part name="U5" library="SparkFun-LED" deviceset="LED-TRICOLOR-5050-IC" device="WS2812-THRU-KIT" value="LED-TRICOLOR-5050-ICWS2812-THRU-KIT"/>
+<part name="U6" library="SparkFun-LED" deviceset="LED-TRICOLOR-5050-IC" device="WS2812-THRU-KIT" value="LED-TRICOLOR-5050-ICWS2812-THRU-KIT"/>
+<part name="U7" library="SparkFun-LED" deviceset="LED-TRICOLOR-5050-IC" device="WS2812-THRU-KIT" value="LED-TRICOLOR-5050-ICWS2812-THRU-KIT"/>
 <part name="GND1" library="SparkFun-Aesthetics" deviceset="GND" device=""/>
 <part name="GND2" library="SparkFun-Aesthetics" deviceset="GND" device=""/>
@@
 <part name="GND15" library="supply1" deviceset="GND" device=""/>
 <part name="JP4" library="SparkFun-Connectors" deviceset="FTDI_BASIC" device="PTH"/>
-<part name="U2" library="SparkFun-LED" deviceset="LED-TRICOLOR-5050-IC" device="WS2812-THRU-KIT" value=""/>
-<part name="U8" library="SparkFun-LED" deviceset="LED-TRICOLOR-5050-IC" device="WS2812-THRU-KIT" value=""/>
-<part name="U9" library="SparkFun-LED" deviceset="LED-TRICOLOR-5050-IC" device="WS2812-THRU-KIT" value=""/>
-<part name="U10" library="SparkFun-LED" deviceset="LED-TRICOLOR-5050-IC" device="WS2812-THRU-KIT" value=""/>
-<part name="U11" library="SparkFun-LED" deviceset="LED-TRICOLOR-5050-IC" device="WS2812-THRU-KIT" value=""/>
+<part name="U2" library="SparkFun-LED" deviceset="LED-TRICOLOR-5050-IC" device="WS2812-THRU-KIT" value="LED-TRICOLOR-5050-ICWS2812-THRU-KIT"/>
+<part name="U8" library="SparkFun-LED" deviceset="LED-TRICOLOR-5050-IC" device="WS2812-THRU-KIT" value="LED-TRICOLOR-5050-ICWS2812-THRU-KIT"/>
+<part name="U9" library="SparkFun-LED" deviceset="LED-TRICOLOR-5050-IC" device="WS2812-THRU-KIT" value="LED-TRICOLOR-5050-ICWS2812-THRU-KIT"/>
+<part name="U10" library="SparkFun-LED" deviceset="LED-TRICOLOR-5050-IC" device="WS2812-THRU-KIT" value="LED-TRICOLOR-5050-ICWS2812-THRU-KIT"/>
+<part name="U11" library="SparkFun-LED" deviceset="LED-TRICOLOR-5050-IC" device="WS2812-THRU-KIT" value="LED-TRICOLOR-5050-ICWS2812-THRU-KIT"/>
 <part name="GND6" library="SparkFun-Aesthetics" deviceset="GND" device=""/>
 <part name="GND12" library="SparkFun-Aesthetics" deviceset="GND" device=""/>
