File: Hardware/ApoBoard_2017_V10.brd (EAGLE design)
At the start: 85.1 x 52.7 mm, 38 parts, among them Q1 RESONATORSMD, U1 PAM2401, U10 LED-TRICOLOR-5050-ICWS2812-TH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, U11 LED-TRICOLOR-5050-ICWS2812-TH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, U13 ATMEGA328, U2 LED-TRICOLOR-5050-ICWS2812-TH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, U3 LED-TRICOLOR-5050-ICWS2812-TH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, U4 LED-TRICOLOR-5050-ICWS2812-TH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, U5 LED-TRICOLOR-5050-ICWS2812-TH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, U6 LED-TRICOLOR-5050-ICWS2812-TH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, U7 LED-TRICOLOR-5050-ICWS2812-TH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, U8 LED-TRICOLOR-5050-ICWS2812-TH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, U9 LED-TRICOLOR-5050-ICWS2812-TH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

Commit message: V1.0 Final version ordered
Parts:
- added TP10, TP7, TP8, TP9: TP-3x5, SparkFun-Passives:PAD.03X.05
- moved U2 0.63 mm to (17.1, -5.08)
- moved U9 0.63 mm to (17.1, 5.08)
Connections:
- removed net N$22: U13.28
- removed net N$23: U13.27
- removed net N$26: U13.24
- removed net N$27: U13.23
- new net N$4: TP7.P$1, U13.27
- new net N$7: TP8.P$1, U13.28
- net +5V: now also TP9.P$1
- net GND: now also TP10.P$1
Routing:
- net N$7: track 0.00 -> 31.8 mm, vias 0 -> 1
- net N$4: track 0.00 -> 29.5 mm, vias 0 -> 1
- net +5V: track 213.8 -> 220.0 mm
Other:
- board text added: "4) Collect as many modes as you can. Press Mode button to cycle through new modes"
- board text added: "A4"
- board text added: "A5"
- board text added: "Joel E B V1.0"
- board text added: "Learn how to hack your eyeball at:"
- board text added: "SCL"
- board text added: "SDA"
- board text removed: "4) Collect as many modes as you can"
- board text removed: "5) Press Mode button to cycle through new modes"
- board text removed: "Joel E B V0.3"
