File: Hardware/ApoBoard_2017_V10.sch (EAGLE design)
At the start: 37 parts, among them Q1 RESONATORSMD, U1 PAM2401, U10 LED-TRICOLOR-5050-ICWS2812-TH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, U11 LED-TRICOLOR-5050-ICWS2812-TH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, U13 ATMEGA328, U2 LED-TRICOLOR-5050-ICWS2812-TH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, U3 LED-TRICOLOR-5050-ICWS2812-TH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, U4 LED-TRICOLOR-5050-ICWS2812-TH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, U5 LED-TRICOLOR-5050-ICWS2812-TH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, U6 LED-TRICOLOR-5050-ICWS2812-TH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

Commit message: V1.0 Final version ordered
Parts:
- added TP10, TP7, TP8, TP9: TP-3x5, SparkFun-Passives:TEST-POINT3X5
Connections:
- removed net N$22: U13.PC5(ADC5/SCL)
- removed net N$23: U13.PC4(ADC4/SDA)
- removed net N$26: U13.PC1(ADC1)
- removed net N$27: U13.PC0(ADC0)
- new net N$4: TP7.1, U13.PC4(ADC4/SDA)
- new net N$7: TP8.1, U13.PC5(ADC5/SCL)
- net +5V: now also TP9.1
- net GND: now also TP10.1
Other:
- note added: "Test Points 7-10: I2C and Analog/Digital Expansion Port"
Changed lines of the file:
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@@
 <part name="BATT1" library="1_BES_ELECTROMECHANICAL" deviceset="BATTERY_HOLDER" device="AA_2466" value="BATTERY_HOLDERAA_2466"/>
 <part name="GND21" library="SparkFun" deviceset="GND" device=""/>
+<part name="TP7" library="SparkFun-Passives" deviceset="TEST-POINT" device="3X5" value="TP-3x5"/>
+<part name="TP8" library="SparkFun-Passives" deviceset="TEST-POINT" device="3X5" value="TP-3x5"/>
+<part name="TP9" library="SparkFun-Passives" deviceset="TEST-POINT" device="3X5" value="TP-3x5"/>
+<part name="TP10" library="SparkFun-Passives" deviceset="TEST-POINT" device="3X5" value="TP-3x5"/>
+<part name="GND17" library="SparkFun" deviceset="GND" device=""/>
+<part name="P+16" library="supply1" deviceset="+5V" device=""/>
 </parts>
 <sheets>
@@
 <text x="172.72" y="81.28" size="2.54" layer="97">ATMEGA328P Programming</text>
 <text x="237.49" y="6.35" size="2.54" layer="94">V0.1</text>
+<text x="116.84" y="48.26" size="1.27" layer="97">Test Points 7-10:
+I2C and Analog/Digital
+Expansion Port</text>
 </plain>
 <instances>
@@
 <attribute name="VALUE" x="27.94" y="40.64" size="1.778" layer="96" rot="R270"/>
 </instance>
+<instance part="TP7" gate="G$1" x="93.98" y="55.88" smashed="yes">
+<attribute name="NAME" x="97.536" y="55.118" size="1.778" layer="95"/>
+</instance>
+<instance part="TP8" gate="G$1" x="93.98" y="53.34" smashed="yes">
+<attribute name="NAME" x="97.536" y="52.578" size="1.778" layer="95"/>
+</instance>
+<instance part="TP9" gate="G$1" x="114.3" y="60.96" smashed="yes">
+<attribute name="NAME" x="117.856" y="60.198" size="1.778" layer="95"/>
+</instance>
+<instance part="TP10" gate="G$1" x="114.3" y="55.88" smashed="yes">
+<attribute name="NAME" x="117.856" y="55.118" size="1.778" layer="95"/>
+</instance>
+<instance part="GND17" gate="1" x="111.76" y="50.8" rot="MR0"/>
+<instance part="P+16" gate="1" x="111.76" y="66.04"/>
 </instances>
 <busses>
@@
 <pinref part="Q1" gate="G$1" pin="2"/>
 <pinref part="GND21" gate="1" pin="GND"/>
+</segment>
+<segment>
+<pinref part="TP10" gate="G$1" pin="1"/>
+<pinref part="GND17" gate="1" pin="GND"/>
+<wire x1="114.3" y1="55.88" x2="111.76" y2="55.88" width="0.1524" layer="91"/>
+<wire x1="111.76" y1="55.88" x2="111.76" y2="53.34" width="0.1524" layer="91"/>
 </segment>
 </net>
@@
 <junction x="93.98" y="121.92"/>
 </segment>
+<segment>
+<pinref part="P+16" gate="1" pin="+5V"/>
+<pinref part="TP9" gate="G$1" pin="1"/>
+<wire x1="111.76" y1="63.5" x2="111.76" y2="60.96" width="0.1524" layer="91"/>
+<wire x1="111.76" y1="60.96" x2="114.3" y2="60.96" width="0.1524" layer="91"/>
+</segment>
 </net>
 <net name="TX" class="0">
@@
 </segment>
 </net>
-<net name="N$22" class="0">
-<segment>
-<wire x1="91.44" y1="53.34" x2="93.98" y2="53.34" width="0.1524" layer="91"/>
-<label x="93.98" y="53.34" size="1.27" layer="95" xref="yes"/>
-<pinref part="U13" gate="G$1" pin="PC5(ADC5/SCL)"/>
-</segment>
-</net>
-<net name="N$23" class="0">
-<segment>
-<wire x1="91.44" y1="55.88" x2="93.98" y2="55.88" width="0.1524" layer="91"/>
-<label x="93.98" y="55.88" size="1.27" layer="95" xref="yes"/>
-<pinref part="U13" gate="G$1" pin="PC4(ADC4/SDA)"/>
-</segment>
-</net>
 <net name="N$24" class="0">
 <segment>
@@
 <label x="93.98" y="60.96" size="1.27" layer="95" xref="yes"/>
 <pinref part="U13" gate="G$1" pin="PC2(ADC2)"/>
-</segment>
-</net>
-<net name="N$26" class="0">
-<segment>
-<wire x1="91.44" y1="63.5" x2="93.98" y2="63.5" width="0.1524" layer="91"/>
-<label x="93.98" y="63.5" size="1.27" layer="95" xref="yes"/>
-<pinref part="U13" gate="G$1" pin="PC1(ADC1)"/>
-</segment>
-</net>
-<net name="N$27" class="0">
-<segment>
-<wire x1="91.44" y1="66.04" x2="93.98" y2="66.04" width="0.1524" layer="91"/>
-<label x="93.98" y="66.04" size="1.27" layer="95" xref="yes"/>
-<pinref part="U13" gate="G$1" pin="PC0(ADC0)"/>
 </segment>
 </net>
@@
 </segment>
 </net>
+<net name="N$4" class="0">
+<segment>
+<pinref part="U13" gate="G$1" pin="PC4(ADC4/SDA)"/>
+<pinref part="TP7" gate="G$1" pin="1"/>
+<wire x1="93.98" y1="55.88" x2="91.44" y2="55.88" width="0.1524" layer="91"/>
+</segment>
+</net>
+<net name="N$7" class="0">
+<segment>
+<pinref part="U13" gate="G$1" pin="PC5(ADC5/SCL)"/>
+<pinref part="TP8" gate="G$1" pin="1"/>
+<wire x1="93.98" y1="53.34" x2="91.44" y2="53.34" width="0.1524" layer="91"/>
+</segment>
+</net>
