File: Testbed/Apo Board 2017_PB_MILLABLE.brd (EAGLE design)
At the start: 201.3 x 74.9 mm, 22 parts, among them J1 AVR_SPI_PROG_3X2PTH, J2 AVR_SPI_PROG_3X2PTH, J3 POWER_JACK

Commit message: Updating Testbed - almost finished
Parts:
- added J9: (no value), SparkFun-Connectors:1X01_LONGPAD
- moved J8 39.6 mm to (17.1, 17.8), turned to 0 degrees
- moved H5 1.27 mm to (-44.5, -29.2)
- moved J1 1.27 mm to (8.89, -39.4)
Connections:
- new net N$16: J8.1, J9.1
- new net N$7: J4.6, J5.1
- new net N$8: J4.5, J5.2
- net GND: no longer J4.5, J4.6, J5.1, J5.2, J8.1
Routing:
- net GND: track 0.00 -> 148.5 mm
- net N$6: track 56.9 -> 0.00 mm
- net N$9: track 55.7 -> 0.00 mm
- net N$12: track 55.7 -> 0.00 mm
- net N$11: track 55.7 -> 0.00 mm
- net N$10: track 55.7 -> 0.00 mm
- net N$16: track 0.00 -> 54.7 mm
- net N$2: track 53.8 -> 0.00 mm
- net N$5: track 52.3 -> 0.00 mm
- net N$3: track 47.0 -> 0.00 mm
- net N$4: track 41.7 -> 0.00 mm
- net N$17: track 49.3 -> 46.4 mm
- removed copper zone on layer 1, net GND
- removed copper zone on layer 16, net GND
Other:
- board text removed: "Analog Meter"
- board text removed: "BLK"
- board text removed: "FTDI"
- board text removed: "GRN"
- board text removed: "PASS"
