File: Testbed/Apo Board 2017_PB_MILLABLE.sch (EAGLE design)
At the start: 22 parts, among them J1 AVR_SPI_PROG_3X2PTH, J2 AVR_SPI_PROG_3X2PTH, J3 POWER_JACK

Commit message: Updating Testbed - almost finished
Parts:
- added J9: (no value), SparkFun-Connectors:CONN_01PTH_LONGPAD
Connections:
- new net N$16: J8.1, J9.1
- new net N$7: J4.6, J5.1
- new net N$8: J4.5, J5.2
- net GND: no longer J4.5, J4.6, J5.1, J5.2, J8.1
Other:
- moved on the sheet: J4, J5, J8
Changed lines of the file:
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@@
 <part name="J7" library="SparkFun-Connectors" deviceset="CONN_01" device="PTH_LONGPAD"/>
 <part name="J8" library="SparkFun-Connectors" deviceset="CONN_01" device="PTH_LONGPAD"/>
+<part name="J9" library="SparkFun-Connectors" deviceset="CONN_01" device="PTH_LONGPAD"/>
 <part name="J10" library="SparkFun-Connectors" deviceset="CONN_01" device="PTH_LONGPAD"/>
 <part name="J11" library="SparkFun-Connectors" deviceset="CONN_01" device="PTH_LONGPAD"/>
@@
 <part name="J13" library="SparkFun-Connectors" deviceset="CONN_01" device="PTH_LONGPAD"/>
 <part name="J14" library="SparkFun-Connectors" deviceset="CONN_01" device="PTH_LONGPAD"/>
-<part name="GND2" library="SparkFun-Aesthetics" deviceset="GND" device=""/>
-<part name="GND4" library="SparkFun-Aesthetics" deviceset="GND" device=""/>
 </parts>
 <sheets>
@@
 <instance part="H5" gate="G$1" x="228.6" y="43.18"/>
 <instance part="H6" gate="G$1" x="236.22" y="43.18"/>
-<instance part="J4" gate="G$1" x="63.5" y="157.48" rot="R180"/>
-<instance part="J5" gate="G$1" x="38.1" y="154.94"/>
+<instance part="J4" gate="G$1" x="40.64" y="154.94"/>
+<instance part="J5" gate="G$1" x="66.04" y="157.48" rot="R180"/>
 <instance part="J6" gate="G$1" x="106.68" y="162.56"/>
 <instance part="J7" gate="G$1" x="129.54" y="162.56" rot="R180"/>
-<instance part="J8" gate="G$1" x="104.14" y="119.38"/>
+<instance part="J8" gate="G$1" x="104.14" y="139.7"/>
+<instance part="J9" gate="G$1" x="129.54" y="139.7" rot="R180"/>
 <instance part="J10" gate="G$1" x="43.18" y="99.06" rot="R180"/>
 <instance part="J11" gate="G$1" x="38.1" y="91.44" rot="R180"/>
@@
 <instance part="J13" gate="G$1" x="104.14" y="129.54"/>
 <instance part="J14" gate="G$1" x="129.54" y="129.54" rot="R180"/>
-<instance part="GND2" gate="1" x="114.3" y="114.3"/>
-<instance part="GND4" gate="1" x="50.8" y="144.78"/>
 </instances>
 <busses>
@@
 <wire x1="185.42" y1="139.7" x2="185.42" y2="137.16" width="0.1524" layer="91"/>
 </segment>
-<segment>
-<pinref part="GND2" gate="1" pin="GND"/>
-<pinref part="J8" gate="G$1" pin="1"/>
-<wire x1="114.3" y1="116.84" x2="114.3" y2="119.38" width="0.1524" layer="91"/>
-<wire x1="114.3" y1="119.38" x2="111.76" y2="119.38" width="0.1524" layer="91"/>
-</segment>
-<segment>
-<pinref part="J4" gate="G$1" pin="6"/>
-<pinref part="J5" gate="G$1" pin="1"/>
-<wire x1="43.18" y1="149.86" x2="48.26" y2="149.86" width="0.1524" layer="91"/>
-<pinref part="GND4" gate="1" pin="GND"/>
-<wire x1="48.26" y1="149.86" x2="50.8" y2="149.86" width="0.1524" layer="91"/>
-<wire x1="50.8" y1="149.86" x2="58.42" y2="149.86" width="0.1524" layer="91"/>
-<wire x1="50.8" y1="147.32" x2="50.8" y2="149.86" width="0.1524" layer="91"/>
-<junction x="50.8" y="149.86"/>
-<pinref part="J4" gate="G$1" pin="5"/>
-<pinref part="J5" gate="G$1" pin="2"/>
-<wire x1="43.18" y1="152.4" x2="48.26" y2="152.4" width="0.1524" layer="91"/>
-<wire x1="48.26" y1="152.4" x2="58.42" y2="152.4" width="0.1524" layer="91"/>
-<wire x1="48.26" y1="149.86" x2="48.26" y2="152.4" width="0.1524" layer="91"/>
-<junction x="48.26" y="149.86"/>
-<junction x="48.26" y="152.4"/>
-</segment>
 </net>
 <net name="N$2" class="0">
@@
 </segment>
 </net>
+<net name="N$7" class="0">
+<segment>
+<pinref part="J4" gate="G$1" pin="6"/>
+<pinref part="J5" gate="G$1" pin="1"/>
+<wire x1="60.96" y1="162.56" x2="45.72" y2="162.56" width="0.1524" layer="91"/>
+</segment>
+</net>
+<net name="N$8" class="0">
+<segment>
+<pinref part="J4" gate="G$1" pin="5"/>
+<pinref part="J5" gate="G$1" pin="2"/>
+<wire x1="60.96" y1="160.02" x2="45.72" y2="160.02" width="0.1524" layer="91"/>
+</segment>
+</net>
 <net name="N$9" class="0">
 <segment>
 <pinref part="J4" gate="G$1" pin="4"/>
 <pinref part="J5" gate="G$1" pin="3"/>
-<wire x1="43.18" y1="154.94" x2="58.42" y2="154.94" width="0.1524" layer="91"/>
+<wire x1="60.96" y1="157.48" x2="45.72" y2="157.48" width="0.1524" layer="91"/>
 </segment>
 </net>
@@
 <pinref part="J4" gate="G$1" pin="3"/>
 <pinref part="J5" gate="G$1" pin="4"/>
-<wire x1="43.18" y1="157.48" x2="58.42" y2="157.48" width="0.1524" layer="91"/>
+<wire x1="60.96" y1="154.94" x2="45.72" y2="154.94" width="0.1524" layer="91"/>
 </segment>
 </net>
@@
 <pinref part="J4" gate="G$1" pin="2"/>
 <pinref part="J5" gate="G$1" pin="5"/>
-<wire x1="43.18" y1="160.02" x2="58.42" y2="160.02" width="0.1524" layer="91"/>
+<wire x1="60.96" y1="152.4" x2="45.72" y2="152.4" width="0.1524" layer="91"/>
 </segment>
 </net>
@@
 <pinref part="J4" gate="G$1" pin="1"/>
 <pinref part="J5" gate="G$1" pin="6"/>
-<wire x1="43.18" y1="162.56" x2="58.42" y2="162.56" width="0.1524" layer="91"/>
+<wire x1="60.96" y1="149.86" x2="45.72" y2="149.86" width="0.1524" layer="91"/>
 </segment>
 </net>
@@
 </segment>
 </net>
+<net name="N$16" class="0">
+<segment>
+<pinref part="J9" gate="G$1" pin="1"/>
+<pinref part="J8" gate="G$1" pin="1"/>
+<wire x1="111.76" y1="139.7" x2="121.92" y2="139.7" width="0.1524" layer="91"/>
+</segment>
+</net>
