File: Testbed/Apo Board 2017_PM.brd (EAGLE design)
At the start: 201.3 x 74.9 mm, 22 parts, among them J1 AVR_SPI_PROG_3X2PTH, J2 AVR_SPI_PROG_3X2PTH, J3 POWER_JACK

Commit message: Updating Testbed - almost finished
Parts:
- removed D1: (no value), SparkFun-LED:LED_5MM
- removed H1, H6: STAND-OFF, SparkFun-Hardware:STAND-OFF
- removed J2: AVR_SPI_PROG_3X2PTH, SparkFun-Connectors:2X3
- removed R1: (no value), SparkFun-Resistors:AXIAL-0.3-KIT
- added J9: (no value), SparkFun-Connectors:1X01_POGOPIN_HOLE_0.58_DIA
- J1: value AVR_SPI_PROG_3X2PTH -> (none); device SparkFun-Connectors:2X3 -> SparkFun-Connectors:1X01_POGOPIN_HOLE_0.58_DIA
- J10, J11, J12, J13, J14, J6, J7, J8: device SparkFun-Connectors:1X01_LONGPAD -> SparkFun-Connectors:1X01_POGOPIN_HOLE_0.58_DIA
- J3: value POWER_JACK -> (none); device SparkFun-Connectors:POWER_JACK_PTH -> SparkFun-Connectors:1X01_POGOPIN_HOLE_0.58_DIA
- J4: device SparkFun-Connectors:1X06_LONGPADS -> SparkFun-Connectors:1X06_HOLES_ONLY
- J5: device SparkFun-Connectors:1X06_LONGPADS -> SparkFun-Connectors:1X01_POGOPIN_HOLE_0.58_DIA
- moved J3 52.9 mm to (0.00, -1.27), turned to 90 degrees
- moved J14 46.0 mm to (-2.54, 1.27)
- moved J8 42.8 mm to (2.54, 1.27)
- moved J5 40.4 mm to (2.54, -1.27), turned to 90 degrees
- moved J1 38.6 mm to (-2.54, -1.27), turned to 90 degrees
- moved FRAME1 9.84 mm to (-26.7, -48.3)
Connections:
- removed net GND: D1.K, J1.6, J11.1, J2.6, J3.GND, J3.GNDBREAK, J4.5, J4.6, J5.1, J5.2, J8.1
- removed net N$1: J10.1, J3.PWR
- removed net N$10: J4.3, J5.4
- removed net N$11: J4.2, J5.5
- removed net N$12: J4.1, J5.6
- removed net N$14: D1.A, R1.P$1
- removed net N$2: J1.4, J2.4
- removed net N$3: J1.2, J2.2
- removed net N$4: J1.5, J2.5
- removed net N$5: J1.3, J2.3
- removed net N$6: J1.1, J2.1
- removed net N$9: J4.4, J5.3
- net N$15: no longer R1.P$2
- net N$17: no longer J14.1
Routing:
- net N$15: track 96.3 -> 0.00 mm
- net N$6: track 56.9 -> 0.00 mm
- net N$9: track 55.7 -> 0.00 mm
- net N$12: track 55.7 -> 0.00 mm
- net N$11: track 55.7 -> 0.00 mm
- net N$10: track 55.7 -> 0.00 mm
- net N$2: track 53.8 -> 0.00 mm
- net N$5: track 52.3 -> 0.00 mm
- net N$17: track 49.3 -> 0.00 mm
- net N$3: track 47.0 -> 0.00 mm
- net N$4: track 41.7 -> 0.00 mm
- net N$1: track 33.6 -> 0.00 mm
- net N$14: track 8.15 -> 0.00 mm
- net N$13: track 2.83 -> 0.00 mm
- removed copper zone on layer 1, net GND
- removed copper zone on layer 16, net GND
Other:
- board size 201.3 x 74.9 mm -> 96.5 x 62.2 mm
- board text removed: "1.5V IN"
- board text removed: "Analog Meter"
- board text removed: "BLK"
- board text removed: "FTDI"
- board text removed: "GRN"
- board text removed: "PASS"
- board text removed: "ROUTE OUT"
