File: Hardware/Testbed/Apo Board 2017_PM.sch (EAGLE design)
At the start: 18 parts

Commit message: Pogo Bed finished.
Finished making pogoed programming and testing fixture. Moving to
Hardware Folder
Parts:
- removed H2, H3, H4, H5: STAND-OFF, SparkFun-Hardware:STAND-OFF
- added J15, J16, J17, J2: (no value), SparkFun-Connectors:CONN_01POGOPIN_HOLE_0.58
Connections:
- removed net N$13: J6.1, J7.1
- removed net N$15: J12.1
- removed net N$17: J13.1
Changed lines of the file:
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@@
 </classes>
 <parts>
-<part name="H2" library="SparkFun-Hardware" deviceset="STAND-OFF" device=""/>
-<part name="H3" library="SparkFun-Hardware" deviceset="STAND-OFF" device=""/>
-<part name="H4" library="SparkFun-Hardware" deviceset="STAND-OFF" device=""/>
-<part name="H5" library="SparkFun-Hardware" deviceset="STAND-OFF" device=""/>
 <part name="J4" library="SparkFun-Connectors" deviceset="CONN_06" device="POGOPIN_HOLES_ONLY"/>
 <part name="J6" library="SparkFun-Connectors" deviceset="CONN_01" device="POGOPIN_HOLE_0.58"/>
@@
 <part name="J9" library="SparkFun-Connectors" deviceset="CONN_01" device="POGOPIN_HOLE_0.58"/>
 <part name="J14" library="SparkFun-Connectors" deviceset="CONN_01" device="POGOPIN_HOLE_0.58"/>
+<part name="J2" library="SparkFun-Connectors" deviceset="CONN_01" device="POGOPIN_HOLE_0.58"/>
+<part name="J15" library="SparkFun-Connectors" deviceset="CONN_01" device="POGOPIN_HOLE_0.58"/>
+<part name="J16" library="SparkFun-Connectors" deviceset="CONN_01" device="POGOPIN_HOLE_0.58"/>
+<part name="J17" library="SparkFun-Connectors" deviceset="CONN_01" device="POGOPIN_HOLE_0.58"/>
 </parts>
 <sheets>
@@
 </plain>
 <instances>
-<instance part="H2" gate="G$1" x="200.66" y="43.18"/>
-<instance part="H3" gate="G$1" x="208.28" y="43.18"/>
-<instance part="H4" gate="G$1" x="218.44" y="43.18"/>
-<instance part="H5" gate="G$1" x="228.6" y="43.18"/>
 <instance part="J4" gate="G$1" x="63.5" y="157.48" rot="R180"/>
 <instance part="J6" gate="G$1" x="106.68" y="162.56"/>
@@
 <instance part="J9" gate="G$1" x="91.44" y="48.26" rot="R180"/>
 <instance part="J14" gate="G$1" x="91.44" y="58.42" rot="R180"/>
+<instance part="J2" gate="G$1" x="167.64" y="91.44" rot="R180"/>
+<instance part="J15" gate="G$1" x="167.64" y="78.74" rot="R180"/>
+<instance part="J16" gate="G$1" x="167.64" y="66.04" rot="R180"/>
+<instance part="J17" gate="G$1" x="167.64" y="53.34" rot="R180"/>
 </instances>
 <busses>
 </busses>
 <nets>
-<net name="N$13" class="0">
-<segment>
-<pinref part="J7" gate="G$1" pin="1"/>
-<pinref part="J6" gate="G$1" pin="1"/>
-<wire x1="114.3" y1="162.56" x2="121.92" y2="162.56" width="0.1524" layer="91"/>
-</segment>
-</net>
-<net name="N$15" class="0">
-<segment>
-<pinref part="J12" gate="G$1" pin="1"/>
-<wire x1="157.48" y1="139.7" x2="160.02" y2="139.7" width="0.1524" layer="91"/>
-</segment>
-</net>
-<net name="N$17" class="0">
-<segment>
-<pinref part="J13" gate="G$1" pin="1"/>
-<wire x1="111.76" y1="129.54" x2="121.92" y2="129.54" width="0.1524" layer="91"/>
-</segment>
-</net>
 </nets>
 </sheet>
