File: Hardware/Testbed/Apo Board 2017_PB.brd (EAGLE design)
At the start: 201.3 x 74.9 mm, 22 parts, among them J1 AVR_SPI_PROG_3X2PTH, J2 AVR_SPI_PROG_3X2PTH, J3 POWER_JACK

Commit message: Pogo Bed finished.
Finished making pogoed programming and testing fixture. Moving to
Hardware Folder
Parts:
- added U6, U7: (no value), SparkFun-LED:LED-RGB-THRU-KIT
Connections:
- new net N$16: U6.1, U7.1
- new net N$18: U6.2, U7.2
- new net N$7: U6.4, U7.4
- net GND: now also U6.3, U7.3
Routing:
- net N$18: track 0.00 -> 36.0 mm
- net N$7: track 0.00 -> 35.2 mm
- net N$16: track 0.00 -> 34.9 mm
Other:
- board size 201.3 x 74.9 mm -> 96.5 x 74.9 mm
- board text removed: "ROUTE OUT"
Changed lines of the file:
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@@
 <layer number="49" name="Reference" color="13" fill="1" visible="no" active="yes"/>
 <layer number="50" name="dxf" color="7" fill="1" visible="no" active="yes"/>
-<layer number="51" name="tDocu" color="6" fill="1" visible="yes" active="yes"/>
+<layer number="51" name="tDocu" color="6" fill="1" visible="no" active="yes"/>
 <layer number="52" name="bDocu" color="7" fill="1" visible="no" active="yes"/>
 <layer number="53" name="tGND_GNDA" color="7" fill="9" visible="no" active="no"/>
@@
 <circle x="0" y="-1.27" radius="1.27" width="0.4064" layer="51"/>
 <circle x="-2.54" y="-1.27" radius="1.27" width="0.4064" layer="51"/>
-<wire x1="-48.26" y1="30.48" x2="48.26" y2="30.48" width="0.2032" layer="20"/>
-<wire x1="48.26" y1="30.48" x2="48.26" y2="-44.45" width="0.2032" layer="20"/>
-<wire x1="48.26" y1="-44.45" x2="-48.26" y2="-44.45" width="0.2032" layer="20"/>
-<wire x1="-48.26" y1="-44.45" x2="-48.26" y2="30.48" width="0.2032" layer="20"/>
-<wire x1="67.9958" y1="-6.2992" x2="153.0858" y2="-6.2992" width="0" layer="20" curve="-127.037923"/>
-<wire x1="153.0858" y1="-6.2992" x2="67.9958" y2="-6.2992" width="0" layer="20" curve="-127.037923"/>
-<text x="107.442" y="0" size="0.9398" layer="51" font="vector" ratio="15" rot="MR90" align="bottom-right">MISO</text>
-<text x="107.315" y="-9.017" size="0.9398" layer="51" font="vector" ratio="15" rot="MR90" align="bottom-right">5V</text>
-<text x="109.982" y="-0.889" size="0.9398" layer="51" font="vector" ratio="15" rot="MR90" align="bottom-right">SCK</text>
-<text x="109.982" y="-9.017" size="0.9398" layer="51" font="vector" ratio="15" rot="MR90" align="bottom-right">MOSI</text>
-<text x="112.522" y="-0.889" size="0.9398" layer="51" font="vector" ratio="15" rot="MR90" align="bottom-right">RST</text>
-<text x="112.522" y="-9.017" size="0.9398" layer="51" font="vector" ratio="15" rot="MR90" align="bottom-right">GND</text>
-<text x="111.125" y="6.858" size="0.9398" layer="51" font="vector" ratio="15" rot="MR90" align="bottom-right">5V</text>
-<text x="106.1085" y="6.9215" size="0.9398" layer="51" font="vector" ratio="15" rot="MR90" align="bottom-right">TX</text>
-<text x="108.6485" y="6.9215" size="0.9398" layer="51" font="vector" ratio="15" rot="MR90" align="bottom-right">RX</text>
-<text x="103.632" y="5.207" size="0.9398" layer="51" font="vector" ratio="15" rot="MR90">DTR</text>
-<text x="113.792" y="7.493" size="0.9398" layer="51" font="vector" ratio="15" rot="MR90" align="bottom-right">GND</text>
-<text x="116.332" y="7.493" size="0.9398" layer="51" font="vector" ratio="15" rot="MR90" align="bottom-right">GND</text>
-<wire x1="106.68" y1="-31.115" x2="114.046" y2="-31.1785" width="0" layer="20" curve="24.10157"/>
-<wire x1="106.68" y1="-31.115" x2="106.045" y2="-29.845" width="0" layer="20" curve="-102.768742"/>
-<wire x1="106.045" y1="-29.845" x2="107.1245" y2="-29.337" width="0" layer="20" curve="-93.491466"/>
-<wire x1="107.1245" y1="-29.337" x2="113.7285" y2="-29.464" width="0" layer="20" curve="32.696336"/>
-<wire x1="114.046" y1="-31.1785" x2="114.1095" y2="-29.337" width="0" layer="20" curve="171.428769"/>
-<wire x1="114.1095" y1="-29.337" x2="113.7285" y2="-29.464" width="0" layer="20" curve="24.932354"/>
-<text x="107.2515" y="-30.9245" size="0.8128" layer="20" font="vector" ratio="15">ROUTE OUT</text>
-<wire x1="114.3" y1="18.415" x2="106.934" y2="18.4785" width="0" layer="20" curve="24.10157"/>
-<wire x1="114.3" y1="18.415" x2="114.935" y2="17.145" width="0" layer="20" curve="-102.768742"/>
-<wire x1="114.935" y1="17.145" x2="113.8555" y2="16.637" width="0" layer="20" curve="-93.491466"/>
-<wire x1="113.8555" y1="16.637" x2="107.2515" y2="16.764" width="0" layer="20" curve="32.696336"/>
-<wire x1="106.934" y1="18.4785" x2="106.8705" y2="16.637" width="0" layer="20" curve="171.428769"/>
-<wire x1="106.8705" y1="16.637" x2="107.2515" y2="16.764" width="0" layer="20" curve="24.932354"/>
-<text x="113.7285" y="18.2245" size="0.8128" layer="20" font="vector" ratio="15" rot="R180">ROUTE OUT</text>
-<text x="125.603" y="9.271" size="0.9398" layer="51" font="vector" ratio="15" rot="MR270" align="bottom-right">A4</text>
-<text x="123.063" y="9.906" size="0.9398" layer="51" font="vector" ratio="15" rot="MR270" align="bottom-right">A5</text>
-<circle x="127.635" y="11.43" radius="0.635" width="0.254" layer="51"/>
-<circle x="125.095" y="12.065" radius="0.635" width="0.254" layer="51"/>
-<circle x="122.555" y="12.7" radius="0.635" width="0.254" layer="51"/>
-<circle x="120.015" y="13.335" radius="0.635" width="0.254" layer="51"/>
-<circle x="85.09" y="-6.604" radius="0.803215625" width="0.254" layer="51"/>
-<circle x="135.89" y="-6.604" radius="0.772509375" width="0.254" layer="51"/>
-<circle x="104.14" y="3.3655" radius="1.08694375" width="0.254" layer="51"/>
-<circle x="106.68" y="3.3655" radius="1.08694375" width="0.254" layer="51"/>
-<circle x="109.22" y="3.3655" radius="1.08694375" width="0.254" layer="51"/>
-<circle x="111.76" y="3.3655" radius="1.08694375" width="0.254" layer="51"/>
-<circle x="114.3" y="3.3655" radius="1.08694375" width="0.254" layer="51"/>
-<circle x="116.84" y="3.3655" radius="1.08694375" width="0.254" layer="51"/>
-<circle x="107.95" y="-5.08" radius="0.635" width="0.254" layer="51"/>
-<circle x="110.49" y="-5.08" radius="0.635" width="0.254" layer="51"/>
-<circle x="113.03" y="-5.08" radius="0.635" width="0.254" layer="51"/>
-<circle x="113.03" y="-7.62" radius="0.635" width="0.254" layer="51"/>
-<circle x="110.49" y="-7.62" radius="0.635" width="0.254" layer="51"/>
-<circle x="107.95" y="-7.62" radius="0.635" width="0.254" layer="51"/>
-<text x="128.143" y="12.446" size="0.9398" layer="51" font="vector" ratio="15" rot="MR270" align="bottom-right">GND</text>
-<text x="125.603" y="13.081" size="0.9398" layer="51" font="vector" ratio="15" rot="MR270" align="bottom-right">SDA</text>
-<text x="123.063" y="13.716" size="0.9398" layer="51" font="vector" ratio="15" rot="MR270" align="bottom-right">SCL</text>
-<text x="119.507" y="16.002" size="0.9398" layer="51" font="vector" ratio="15" rot="MR90" align="bottom-right">5V</text>
-<circle x="129.3622" y="-22.7076" radius="1.1447625" width="0.254" layer="51"/>
-<circle x="131.45135" y="-20.96135" radius="1.1447625" width="0.254" layer="51"/>
-<wire x1="84.455" y1="-3.81" x2="85.725" y2="-3.81" width="0.254" layer="51"/>
-<wire x1="135.255" y1="-3.81" x2="136.525" y2="-3.81" width="0.254" layer="51"/>
-<wire x1="135.89" y1="-3.175" x2="135.89" y2="-4.445" width="0.254" layer="51"/>
+<wire x1="-48.26" y1="30.48" x2="48.26" y2="30.48" width="0" layer="20"/>
+<wire x1="48.26" y1="30.48" x2="48.26" y2="-44.45" width="0" layer="20"/>
+<wire x1="48.26" y1="-44.45" x2="-48.26" y2="-44.45" width="0" layer="20"/>
+<wire x1="-48.26" y1="-44.45" x2="-48.26" y2="30.48" width="0" layer="20"/>
 <text x="-3.048" y="6.35" size="0.9398" layer="51" font="vector" ratio="15" rot="MR90" align="bottom-right">MISO</text>
 <text x="-3.175" y="-2.667" size="0.9398" layer="51" font="vector" ratio="15" rot="MR90" align="bottom-right">5V</text>
@@
 <text x="-3.302" y="-42.545" size="1.4224" layer="21" font="vector" ratio="15" rot="R90">BLK</text>
 <text x="33.02" y="-8.255" size="1.4224" layer="21" font="vector" ratio="15">Analog Meter</text>
+<wire x1="-42.4942" y1="0.0508" x2="42.5958" y2="0.0508" width="0" layer="51" curve="-127.037923"/>
+<wire x1="42.5958" y1="0.0508" x2="-42.4942" y2="0.0508" width="0" layer="51" curve="-127.037923"/>
+<circle x="-2.413" y="-17.0942" radius="0.568278125" width="0.254" layer="51"/>
+<circle x="0.635" y="-17.10055" radius="0.568278125" width="0.254" layer="51"/>
+<circle x="-0.89535" y="-17.41805" radius="0.568278125" width="0.254" layer="51"/>
+<circle x="2.159" y="-17.41805" radius="0.568278125" width="0.254" layer="51"/>
 </plain>
 <attributes>
@@
 <element name="J13" library="SparkFun-Connectors" package="1X01_LONGPAD" value="" x="9.525" y="19.685"/>
 <element name="J14" library="SparkFun-Connectors" package="1X01_LONGPAD" value="" x="43.18" y="-3.81" rot="R90"/>
+<element name="U6" library="SparkFun-LED" package="LED-RGB-THRU-KIT" value="" x="0" y="-16.891" rot="R180"/>
+<element name="U7" library="SparkFun-LED" package="LED-RGB-THRU-KIT" value="" x="-25.4" y="-30.48" rot="R180"/>
 </elements>
 <signals>
@@
 <contactref element="J4" pad="5"/>
 <contactref element="J5" pad="2"/>
+<contactref element="U7" pad="3"/>
+<contactref element="U6" pad="3"/>
 </signal>
 <signal name="N$2">
@@
 <wire x1="43.18" y1="0" x2="43.18" y2="-3.81" width="1.27" layer="1"/>
 </signal>
+<signal name="N$7">
+<contactref element="U6" pad="4"/>
+<contactref element="U7" pad="4"/>
+<wire x1="2.159" y1="-17.4149" x2="2.159" y2="-24.511" width="0.4064" layer="1"/>
+<wire x1="2.159" y1="-24.511" x2="-3.81" y2="-30.48" width="0.4064" layer="1"/>
+<wire x1="-3.81" y1="-30.48" x2="-22.7171" y2="-30.48" width="0.4064" layer="1"/>
+<wire x1="-22.7171" y1="-30.48" x2="-23.241" y2="-31.0039" width="0.4064" layer="1"/>
+</signal>
+<signal name="N$16">
+<contactref element="U6" pad="1"/>
+<contactref element="U7" pad="1"/>
+<wire x1="-2.413" y1="-17.0974" x2="-20.9074" y2="-17.0974" width="0.4064" layer="1"/>
+<wire x1="-20.9074" y1="-17.0974" x2="-27.813" y2="-24.003" width="0.4064" layer="1"/>
+<wire x1="-27.813" y1="-24.003" x2="-27.813" y2="-30.6864" width="0.4064" layer="1"/>
+</signal>
+<signal name="N$18">
+<contactref element="U6" pad="2"/>
+<contactref element="U7" pad="2"/>
+<wire x1="-26.289" y1="-31.0039" x2="-26.289" y2="-25.019" width="0.4064" layer="1"/>
+<wire x1="-26.289" y1="-25.019" x2="-25.4" y2="-24.13" width="0.4064" layer="1"/>
+<wire x1="-25.4" y1="-24.13" x2="-5.08" y2="-24.13" width="0.4064" layer="1"/>
+<wire x1="-5.08" y1="-24.13" x2="-0.889" y2="-19.939" width="0.4064" layer="1"/>
+<wire x1="-0.889" y1="-19.939" x2="-0.889" y2="-17.4149" width="0.4064" layer="1"/>
+</signal>
 </signals>

Commit message: refining bottom layer of testbed
Parts:
- D1: device SparkFun-LED:LED_5MM -> SparkFun-LED:LED5MM
- U6, U7: value (none) -> LED-TRICOLOR-5050-ICWS2812; device SparkFun-LED:LED-RGB-THRU-KIT -> SparkFun-LED:LED-WS2812-THRU
Changed lines of the file:
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@@
 <layer number="47" name="Measures" color="7" fill="1" visible="no" active="yes"/>
 <layer number="48" name="Document" color="7" fill="1" visible="no" active="yes"/>
-<layer number="49" name="Reference" color="13" fill="1" visible="no" active="yes"/>
+<layer number="49" name="Reference" color="13" fill="1" visible="yes" active="yes"/>
 <layer number="50" name="dxf" color="7" fill="1" visible="no" active="yes"/>
-<layer number="51" name="tDocu" color="6" fill="1" visible="no" active="yes"/>
+<layer number="51" name="tDocu" color="6" fill="1" visible="yes" active="yes"/>
 <layer number="52" name="bDocu" color="7" fill="1" visible="no" active="yes"/>
 <layer number="53" name="tGND_GNDA" color="7" fill="9" visible="no" active="no"/>
@@
 <element name="J10" library="SparkFun-Connectors" package="1X01_LONGPAD" value="" x="25.4" y="-0.254"/>
 <element name="J11" library="SparkFun-Connectors" package="1X01_LONGPAD" value="" x="-25.4" y="-0.254"/>
-<element name="D1" library="SparkFun-LED" package="LED_5MM" value="" x="-33.02" y="-38.1"/>
+<element name="D1" library="SparkFun-LED" package="LED5MM" value="" x="-33.02" y="-38.1"/>
 <element name="R1" library="SparkFun-Resistors" package="AXIAL-0.3-KIT" value=" " x="-35.56" y="-26.67" rot="R90">
 <attribute name="PROD_ID" value=" " x="-35.56" y="-26.67" size="1.778" layer="27" font="vector" ratio="15" rot="R90" display="off"/>
@@
 <element name="J13" library="SparkFun-Connectors" package="1X01_LONGPAD" value="" x="9.525" y="19.685"/>
 <element name="J14" library="SparkFun-Connectors" package="1X01_LONGPAD" value="" x="43.18" y="-3.81" rot="R90"/>
-<element name="U6" library="SparkFun-LED" package="LED-RGB-THRU-KIT" value="" x="0" y="-16.891" rot="R180"/>
-<element name="U7" library="SparkFun-LED" package="LED-RGB-THRU-KIT" value="" x="-25.4" y="-30.48" rot="R180"/>
+<element name="U6" library="SparkFun-LED" package="LED-WS2812-THRU" value="LED-TRICOLOR-5050-ICWS2812" x="0" y="-16.891" rot="R180"/>
+<element name="U7" library="SparkFun-LED" package="LED-WS2812-THRU" value="LED-TRICOLOR-5050-ICWS2812" x="-25.4" y="-30.48" rot="R180"/>
 </elements>
 <signals>
